Commit message: PAdded table and primitive gripper in simulation

File: schunk_gripper_communication/urdf/lwa4p/arm.urdf (robot description, URDF)
Before this commit: robot arm, 10 links, 8 joints
Links:
- added link camera_link, mass 10; collision mesh filename=package://schunk_gripper_communication/meshes/cylinder-noto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 scale=1.85 0.2 1.85; visual mesh filename=package://schunk_gripper_communication/meshes/cylinder-noto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 scale=1.85 0.2 1.85
- added link gripper_link, mass 0.5; collision box size=0.1 0.1 0.13; visual box size=0.1 0.1 0.13
- link table_link: geometry collision cylinder length=0.01 radius=0.9; visual cylinder length=0.01 radius=0.9
Joints:
- added joint camera_base_joint: type fixed, parent base_link, child camera_link, origin xyz=0 0 0 rpy=0 0 0
- added joint gripper_joint: type fixed, parent arm_6_link, child gripper_link, origin xyz=0 0 0.32 rpy=0 0 0
- added joint table_base_joint: type fixed, parent base_link, child table_link, origin xyz=0 0 0 rpy=0 0 0
- joint arm_0_joint: parent base_link -> table_link
- joint arm_tcp_joint: parent arm_6_link -> gripper_link

File: schunk_gripper_communication/urdf/lwa4p/lwa4p.urdf.xacro (robot description, xacro)
@@ -16,10 +16,4 @@
   <!-- Schunk Powerball (LWA4P) Macro -->
   <xacro:macro name="schunk_lwa4p" params="parent name *origin">
-    <!-- joint between base_link and arm_0_link -->
-    <joint name="${name}_0_joint" type="fixed" >
-      <xacro:insert_block name="origin" />
-      <parent link="${parent}" />
-      <child link="${name}_0_link" />
-    </joint>
     <joint name="table_base_joint" type="fixed" >
       <xacro:insert_block name="origin" />
@@ -27,4 +21,10 @@
       <child link="table_link" />
     </joint>
+<!-- joint between base_link and arm_0_link -->
+    <joint name="${name}_0_joint" type="fixed" >
+      <xacro:insert_block name="origin" />
+      <parent link="table_link" />
+      <child link="${name}_0_link" />
+    </joint>
     <joint name="camera_base_joint" type="fixed" >
       <xacro:insert_block name="origin" />
@@ -59,5 +59,5 @@
       </inertial>
        <visual>
-        <origin xyz="0 0 -0.01" rpy="0 0 0" />
+        <origin xyz="0 0 0" rpy="0 0 0" />
         <geometry>
             <cylinder length="0.01" radius="0.9" />
@@ -66,5 +66,5 @@
       </visual>
       <collision>
-        <origin xyz="0 0 -0.01" rpy="0 0 0" />
+        <origin xyz="0 0 0" rpy="0 0 0" />
         <geometry>
             <cylinder length="0.01" radius="0.9" />
@@ -303,14 +303,14 @@
       </inertial>
        <visual>
-        <origin xyz="0 0 -0.11" rpy="0 0 0" />
-        <geometry>
-            <box size="0.1 0.1 0.25" />
+        <origin xyz="0 0 -0.17" rpy="0 0 0" />
+        <geometry>
+            <box size="0.1 0.1 0.13" />
         </geometry>
         <material name="Schunk/Yellow" />
       </visual>
       <collision>
-        <origin xyz="0 0 -0.11" rpy="0 0 0" />
-        <geometry>
-            <box size="0.1 0.1 0.25" />
+        <origin xyz="0 0 -0.17" rpy="0 0 0" />
+        <geometry>
+            <box size="0.1 0.1 0.13" />
         </geometry>
       </collision>
