Commit message: Added table and primitive for gripper

File: schunk_gripper_communication/urdf/lwa4p/lwa4p.urdf.xacro (robot description, xacro)
@@ -4,7 +4,7 @@
   <xacro:property name="safety_offset" value="0.02"/>
   <!-- Some additional information used by other tools -->
-  <xacro:include filename="$(find schunk_canopen_driver)/urdf/lwa4p/lwa4p.gazebo.xacro" />
-  <xacro:include filename="$(find schunk_canopen_driver)/urdf/lwa4p/lwa4p.transmission.xacro" />
-  <xacro:include filename="$(find schunk_canopen_driver)/urdf/materials.urdf.xacro" />
+  <xacro:include filename="$(find schunk_gripper_communication)/urdf/lwa4p/lwa4p.gazebo.xacro" />
+  <xacro:include filename="$(find schunk_gripper_communication)/urdf/lwa4p/lwa4p.transmission.xacro" />
+  <xacro:include filename="$(find schunk_gripper_communication)/urdf/materials.urdf.xacro" />
   <xacro:macro name="default_inertial" params="mass">
     <inertial>
@@ -22,5 +22,55 @@
       <child link="${name}_0_link" />
     </joint>
-    <link name="${name}_0_link">
+    <joint name="table_base_joint" type="fixed" >
+      <xacro:insert_block name="origin" />
+      <parent link="${parent}" />
+      <child link="table_link" />
+    </joint>
+    <joint name="camera_base_joint" type="fixed" >
+      <xacro:insert_block name="origin" />
+      <parent link="${parent}" />
+      <child link="camera_link" />
+    </joint>
+    <link name="camera_link">
+      <inertial>
+        <origin xyz="0 0 0" rpy="0 0 0" />
+        <mass value="10"/>
+        <inertia ixx="0.01" ixy="0" ixz="0" iyy="0.01" iyz="0" izz="0.01" />
+      </inertial>
+       <visual>
+        <origin xyz="0 0 -0.01" rpy="1.57 0 0" />
+        <geometry>
+          <mesh filename="package://schunk_gripper_communication/meshes/cylinder-notop.dae" scale="1.85 0.2 1.85"/>
+        </geometry>
+        <material name="Schunk/Yellow" />
+      </visual>
+      <collision>
+        <origin xyz="0 0 -0.01" rpy="1.57 0 0" />
+        <geometry>
+          <mesh filename="package://schunk_gripper_communication/meshes/cylinder-notop.dae" scale="1.85 0.2 1.85"/>
+        </geometry>
+      </collision>
+     </link>
+    <link name="table_link">
+      <inertial>
+        <origin xyz="0 0 0" rpy="0 0 0" />
+        <mass value="10"/>
+        <inertia ixx="0.01" ixy="0" ixz="0" iyy="0.01" iyz="0" izz="0.01" />
+      </inertial>
+       <visual>
+        <origin xyz="0 0 -0.01" rpy="0 0 0" />
+        <geometry>
+            <cylinder length="0.01" radius="0.9" />
+        </geometry>
+        <material name="Schunk/Yellow" />
+      </visual>
+      <collision>
+        <origin xyz="0 0 -0.01" rpy="0 0 0" />
+        <geometry>
+            <cylinder length="0.01" radius="0.9" />
+        </geometry>
+      </collision>
+     </link>
+     <link name="${name}_0_link">
       <inertial>
         <origin xyz="0 0 0" rpy="0 0 0" />
@@ -31,12 +81,12 @@
         <origin xyz="0 0 0" rpy="0 0 0" />
         <geometry>
-          <mesh filename="package://schunk_canopen_driver/meshes/lwa4p/arm_0_link.dae" />
-        </geometry>
-        <material name="Schunk/DarkGrey" />
-      </visual>
-      <collision>
-        <origin xyz="0 0 0" rpy="0 0 0" />
-        <geometry>
-          <mesh filename="package://schunk_canopen_driver/meshes/lwa4p/arm_0_link.stl" />
+          <mesh filename="package://schunk_gripper_communication/meshes/lwa4p/arm_0_link.dae" />
+        </geometry>
+        <material name="Schunk/DarkGrey" />
+      </visual>
+      <collision>
+        <origin xyz="0 0 0" rpy="0 0 0" />
+        <geometry>
+          <mesh filename="package://schunk_gripper_communication/meshes/lwa4p/arm_0_link.stl" />
         </geometry>
       </collision>
@@ -62,12 +112,12 @@
         <origin xyz="0 0 0" rpy="0 0 0" />
         <geometry>
-          <mesh filename="package://schunk_canopen_driver/meshes/lwa4p/arm_1_link.dae" />
-        </geometry>
-        <material name="Schunk/DarkGrey" />
-      </visual>
-      <collision>
-        <origin xyz="0 0 0" rpy="0 0 0" />
-        <geometry>
-          <mesh filename="package://schunk_canopen_driver/meshes/lwa4p/arm_1_link.stl" />
+          <mesh filename="package://schunk_gripper_communication/meshes/lwa4p/arm_1_link.dae" />
+        </geometry>
+        <material name="Schunk/DarkGrey" />
+      </visual>
+      <collision>
+        <origin xyz="0 0 0" rpy="0 0 0" />
+        <geometry>
+          <mesh filename="package://schunk_gripper_communication/meshes/lwa4p/arm_1_link.stl" />
         </geometry>
       </collision>
@@ -95,5 +145,5 @@
         <origin xyz="0 0 0" rpy="0 0 0" />
         <geometry>
-          <mesh filename="package://schunk_canopen_driver/meshes/lwa4p/arm_2_link.dae" />
+          <mesh filename="package://schunk_gripper_communication/meshes/lwa4p/arm_2_link.dae" />
         </geometry>
         <material name="Schunk/Blue" />
@@ -102,5 +152,5 @@
         <origin xyz="0 0 0" rpy="0 0 0" />
         <geometry>
-          <mesh filename="package://schunk_canopen_driver/meshes/lwa4p/arm_2_link.stl" />
+          <mesh filename="package://schunk_gripper_communication/meshes/lwa4p/arm_2_link.stl" />
         </geometry>
       </collision>
@@ -127,12 +177,12 @@
         <origin xyz="0 0 0" rpy="0 0 0" />
         <geometry>
-          <mesh filename="package://schunk_canopen_driver/meshes/lwa4p/arm_3_link.dae" />
-        </geometry>
-        <material name="Schunk/DarkGrey" />
-      </visual>
-      <collision>
-        <origin xyz="0 0 0" rpy="0 0 0" />
-        <geometry>
-          <mesh filename="package://schunk_canopen_driver/meshes/lwa4p/arm_3_link.stl" />
+          <mesh filename="package://schunk_gripper_communication/meshes/lwa4p/arm_3_link.dae" />
+        </geometry>
+        <material name="Schunk/DarkGrey" />
+      </visual>
+      <collision>
+        <origin xyz="0 0 0" rpy="0 0 0" />
+        <geometry>
+          <mesh filename="package://schunk_gripper_communication/meshes/lwa4p/arm_3_link.stl" />
         </geometry>
       </collision>
@@ -158,5 +208,5 @@
         <origin xyz="0 0 0" rpy="0 0 0" />
         <geometry>
-          <mesh filename="package://schunk_canopen_driver/meshes/lwa4p/arm_4_link.dae" />
+          <mesh filename="package://schunk_gripper_communication/meshes/lwa4p/arm_4_link.dae" />
         </geometry>
         <material name="Schunk/Blue" />
@@ -165,5 +215,5 @@
         <origin xyz="0 0 0" rpy="0 0 0" />
         <geometry>
-          <mesh filename="package://schunk_canopen_driver/meshes/lwa4p/arm_4_link.stl" />
+          <mesh filename="package://schunk_gripper_communication/meshes/lwa4p/arm_4_link.stl" />
         </geometry>
       </collision>
@@ -189,12 +239,12 @@
         <origin xyz="0 0 0" rpy="0 0 0" />
         <geometry>
-          <mesh filename="package://schunk_canopen_driver/meshes/lwa4p/arm_5_link.dae" />
-        </geometry>
-        <material name="Schunk/DarkGrey" />
-      </visual>
-      <collision>
-        <origin xyz="0 0 0" rpy="0 0 0" />
-        <geometry>
-          <mesh filename="package://schunk_canopen_driver/meshes/lwa4p/arm_5_link.stl" />
+          <mesh filename="package://schunk_gripper_communication/meshes/lwa4p/arm_5_link.dae" />
+        </geometry>
+        <material name="Schunk/DarkGrey" />
+      </visual>
+      <collision>
+        <origin xyz="0 0 0" rpy="0 0 0" />
+        <geometry>
+          <mesh filename="package://schunk_gripper_communication/meshes/lwa4p/arm_5_link.stl" />
         </geometry>
       </collision>
@@ -221,19 +271,53 @@
         <origin xyz="0 0 0" rpy="0 0 0" />
         <geometry>
-          <mesh filename="package://schunk_canopen_driver/meshes/lwa4p/arm_6_link.dae" />
-        </geometry>
-        <material name="Schunk/DarkGrey" />
-      </visual>
-      <collision>
-        <origin xyz="0 0 0" rpy="0 0 0" />
-        <geometry>
-          <mesh filename="package://schunk_canopen_driver/meshes/lwa4p/arm_6_link.stl" />
+          <mesh filename="package://schunk_gripper_communication/meshes/lwa4p/arm_6_link.dae" />
+        </geometry>
+        <material name="Schunk/DarkGrey" />
+      </visual>
+      <collision>
+        <origin xyz="0 0 0" rpy="0 0 0" />
+        <geometry>
+          <mesh filename="package://schunk_gripper_communication/meshes/lwa4p/arm_6_link.stl" />
         </geometry>
       </collision>
     </link>
     <!-- joint between arm_6_link and tcp_link -->
+    <!--<joint name="${name}_tcp_joint" type="fixed">
+      <origin xyz="0 0 0.08" rpy="0 0 0" />
+      <parent link="${name}_6_link"/>
+      <child link="${name}_tcp_link"/>
+    </joint>
+    <link name="${name}_tcp_link">
+    </link>
+    -->
+    <joint name="gripper_joint" type="fixed" >
+        <origin xyz="0 0 0.32" rpy="0 0 0" />
+        <parent link="${name}_6_link" />
+      <child link="gripper_link" />
+    </joint>
+    <link name="gripper_link">
+      <inertial>
+        <origin xyz="0 0 0.13" rpy="0 0 0" />
+        <mass value="0.5"/>
+        <inertia ixx="0.01" ixy="0" ixz="0" iyy="0.01" iyz="0" izz="0.01" />
+      </inertial>
+       <visual>
+        <origin xyz="0 0 -0.11" rpy="0 0 0" />
+        <geometry>
+            <box size="0.1 0.1 0.25" />
+        </geometry>
+        <material name="Schunk/Yellow" />
+      </visual>
+      <collision>
+        <origin xyz="0 0 -0.11" rpy="0 0 0" />
+        <geometry>
+            <box size="0.1 0.1 0.25" />
+        </geometry>
+      </collision>
+     </link>
+<!-- joint between arm_6_link and tcp_link -->
     <joint name="${name}_tcp_joint" type="fixed">
       <origin xyz="0 0 0.08" rpy="0 0 0" />
-      <parent link="${name}_6_link"/>
+      <parent link="gripper_link"/>
       <child link="${name}_tcp_link"/>
     </joint>

File: schunk_gripper_communication/urdf/materials.urdf.xacro (robot description, xacro)
@@ -10,3 +10,6 @@
     <color rgba="0.0 0.0 0.25 1.0"/>
   </material>
+  <material name="Schunk/Yellow">
+    <color rgba="0.25 0.25 0.0 1.0"/>
+  </material>
 </robot>

Commit message: Arm moves to point now

File: schunk_gripper_communication/urdf/lwa4p/lwa4p.urdf.xacro (robot description, xacro)
@@ -292,5 +292,5 @@
     -->
     <joint name="gripper_joint" type="fixed" >
-        <origin xyz="0 0 0.32" rpy="0 0 0" />
+        <origin xyz="0 0 0.27" rpy="0 0 0" />
         <parent link="${name}_6_link" />
       <child link="gripper_link" />
@@ -303,14 +303,14 @@
       </inertial>
        <visual>
-        <origin xyz="0 0 -0.17" rpy="0 0 0" />
-        <geometry>
-            <box size="0.1 0.1 0.13" />
+        <origin xyz="0 0 -0.15" rpy="0 0 0" />
+        <geometry>
+            <box size="0.1 0.1 0.10" />
         </geometry>
         <material name="Schunk/Yellow" />
       </visual>
       <collision>
-        <origin xyz="0 0 -0.17" rpy="0 0 0" />
-        <geometry>
-            <box size="0.1 0.1 0.13" />
+        <origin xyz="0 0 -0.15" rpy="0 0 0" />
+        <geometry>
+            <box size="0.1 0.1 0.10" />
         </geometry>
       </collision>
